File: FC Design/AIS IREC 2026 FC/AIS IREC 2026 FC.kicad_sch (KiCad schematic)
At the start: 50 parts, among them IC1 ADXL314WBCPZ-RL, IC2 MT29F8G08ABACAWP-IT_C_TR, J1 USB4216-03-A, J2 EBAA-02-C, J3 Conn_01x08, J4 EBAA-02-C, J5 EBAA-02-C, Q1 MMBT3906-TP, Q2 DMN2008LFU-7, Q3 DMN2008LFU-7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

Commit message: Readability changes
Connections:
- net 3.3V: now also R5.2; no longer IC1.5 (VS), J3.3 (Pin_3), Q2.1 (S1), Q2.4 (S2), Q3.1 (S1), Q3.4 (S2), R5.1, U1.21 (VREF+), U2.4 (VCC), Y1.4 (VDD)
- net at U1.14 (NRST): now also R5.1; no longer R5.2
- net at U6.32 (RBIAS): now also R1.2; no longer R1.1
- net Capacitor Ground renamed GND
- net GND: now also R1.1; no longer R1.2
- new net Noise Capacitors: IC1.5 (VS), U1.21 (VREF+), U2.4 (VCC), Y1.4 (VDD)
- new net VBAT: J3.3 (Pin_3), Q2.1 (S1), Q2.4 (S2), Q3.1 (S1), Q3.4 (S2)
Other:
- note removed: "Label Connections"
- moved on the sheet: R1, R2, R5
