File: FC Design/AIS IREC 2026 FC/_autosave-AIS IREC 2026 FC.kicad_sch (KiCad schematic)
At the start: 66 parts, among them IC1 ADXL314WBCPZ-RL, IC2 MT29F8G08ABACAWP-IT_C_TR, J1 USB4216-03-A, J2 EBAA-02-C, J3 Conn_01x08, J4 EBAA-02-C, J5 EBAA-02-C, Q1 MMBT3906-TP, Q2 DMN2008LFU-7, Q3 DMN2008LFU-7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

Commit message: Added PCB layout
Layout is 48% smaller than AV bay was designed to hold, so no issues, space left because I'm lazy. Allows for further improvement in subsequent years.
Parts:
- removed C24, C25: 100nF, SamacSys_Parts:GRM022C81C222KE01L, symbol SamacSys_Parts:GRM022R61A104KE01L
- removed LED2, LED3: 598-8D91-127F, SamacSys_Parts:5988D91127F, symbol SamacSys_Parts:598-8D91-127F
- removed R4, R6: 10KR, Resistor_SMD:R_0201_0603Metric, symbol Device:R
